File: Hardware/Joystickv04.brd (EAGLE design)
At the start: 100 x 48.9 mm, 58 parts, among them J1 AVR_SPI_PRG_6PTH, U1 JOYSTICKPTH, U3 V_REG_MIC5219SMD, U4 MCP73831

Commit message: Almost ready for review
Parts:
- U$2: value XBEE-1B1 -> XBEE-1B2; device SparkFun-RF:XBEE-1 -> SparkFun-RF:XBEE-SILK
- moved LOGO1 19.1 mm to (66.0, 32.4)
Routing:
- net USB_VCC: track 216.6 -> 219.3 mm
- net VBATT: track 101.2 -> 102.8 mm
- net N$5: track 10.9 -> 12.2 mm
- net N$29: track 39.7 -> 40.5 mm
Other:
- board text added: "ASO"
- board text added: "Battery"
- board text added: "D2"
- board text added: "D3"
- board text added: "LEDs"
- board text added: "RSSI"
- board text added: "USB Power"

Commit message: Pre-review
V05.  This version has standoffs and is ready for a few comments before
bringing to engineering review
Parts:
- renumbered J1 to AVR_SPI, JP3 to USB_MICROB, U$1 to ATMEGA32U4, U3 to MIC5219
Routing:
- net GND: track 313.6 -> 311.3 mm
- net N$29: track 40.5 -> 38.8 mm
Other:
- board text removed: "I2C"
