File: Hardware/Joystickv05.sch (EAGLE design)
At the start: 58 parts, among them J1 AVR_SPI_PRG_6PTH, U1 JOYSTICKPTH, U3 V_REG_MIC5219SMD, U4 MCP73831

Commit message: Pre-review
V05.  This version has standoffs and is ready for a few comments before
bringing to engineering review
Parts:
- removed J1: AVR_SPI_PRG_6PTH, SparkFun-Connectors:AVR_SPI_PRG_6PTH
- removed JP3: USB_MICROB_PLUGCONN-11752, SparkFun-Connectors:USB_MICROB_PLUGCONN-11752
- removed U$1: ATMEGA32U41:1-LESS_PASTE, SparkFun-DigitalIC:ATMEGA32U41:1-LESS_PASTE
- added ATMEGA32U4: ATMEGA32U41:1-LESS_PASTE, SparkFun-DigitalIC:ATMEGA32U41:1-LESS_PASTE
- added AVR_SPI: AVR_SPI_PRG_6PTH, SparkFun-Connectors:AVR_SPI_PRG_6PTH
- added STANDOFF1, STANDOFF2, STANDOFF3, STANDOFF4: STAND-OFF, SparkFun-Electromechanical:STAND-OFF
- added USB_MICROB: USB_MICROB_PLUGCONN-11752, SparkFun-Connectors:USB_MICROB_PLUGCONN-11752
- U$2: value XBEE-1B1 -> XBEE-1B2; device SparkFun-RF:XBEE-1B1 -> SparkFun-RF:XBEE-1B2
- renumbered U3 to MIC5219
Connections:
- net 3.3V: now also ATMEGA32U4.AVCC@24, ATMEGA32U4.AVCC@44, ATMEGA32U4.VCC@14, ATMEGA32U4.VCC@34, AVR_SPI.2; no longer J1.2, U$1.AVCC@24, U$1.AVCC@44, U$1.VCC@14, U$1.VCC@34
- net A0: now also ATMEGA32U4.PF7(ADC7); no longer U$1.PF7(ADC7)
- net A1: now also ATMEGA32U4.PF6(ADC6); no longer U$1.PF6(ADC6)
- net D+: now also ATMEGA32U4.D+; no longer U$1.D+
- net D-: now also ATMEGA32U4.D-; no longer U$1.D-
- net D10: now also ATMEGA32U4.PB6(ADC13); no longer U$1.PB6(ADC13)
- net D2: now also ATMEGA32U4.PD1(SDA); no longer U$1.PD1(SDA)
- net D3: now also ATMEGA32U4.PD0(SCL); no longer U$1.PD0(SCL)
- net D4: now also ATMEGA32U4.PD4(ADC8); no longer U$1.PD4(ADC8)
- net D5: now also ATMEGA32U4.PC6; no longer U$1.PC6
- net D6: now also ATMEGA32U4.PD7(ADC10); no longer U$1.PD7(ADC10)
- net D7: now also ATMEGA32U4.PE6; no longer U$1.PE6
- net D8: now also ATMEGA32U4.PB4(ADC11); no longer U$1.PB4(ADC11)
- net D9: now also ATMEGA32U4.PB5(ADC12); no longer U$1.PB5(ADC12)
- net GND: now also ATMEGA32U4.GND@15, ATMEGA32U4.GND@23, ATMEGA32U4.GND@35, ATMEGA32U4.GND@43, ATMEGA32U4.PE2/!HWB, ATMEGA32U4.UGND, AVR_SPI.6, USB_MICROB.GND; no longer J1.6, JP3.GND, U$1.GND@15, U$1.GND@23, U$1.GND@35, U$1.GND@43, U$1.PE2/!HWB, U$1.UGND
- net MISO: now also ATMEGA32U4.PB3(MISO), AVR_SPI.1; no longer J1.1, U$1.PB3(MISO)
- net MOSI: now also ATMEGA32U4.PB2(MOSI), AVR_SPI.4; no longer J1.4, U$1.PB2(MOSI)
- net N$1: now also ATMEGA32U4.XTAL1; no longer U$1.XTAL1
- net N$2: now also ATMEGA32U4.AREF; no longer U$1.AREF
- net N$29: now also ATMEGA32U4.PB0(SS); no longer U$1.PB0(SS)
- net N$3: now also USB_MICROB.D+; no longer JP3.D+
- net N$32: now also ATMEGA32U4.PD5; no longer U$1.PD5
- net N$5: now also ATMEGA32U4.UCAP; no longer U$1.UCAP
- net N$6: now also ATMEGA32U4.XTAL2; no longer U$1.XTAL2
- net N$9: now also USB_MICROB.D-; no longer JP3.D-
- net RESET: now also ATMEGA32U4.!RESET, AVR_SPI.5; no longer J1.5, U$1.!RESET
- net RX: now also ATMEGA32U4.PD2(RX); no longer U$1.PD2(RX)
- net SCK: now also ATMEGA32U4.PB1(SCK), AVR_SPI.3; no longer J1.3, U$1.PB1(SCK)
- net TX: now also ATMEGA32U4.PD3(TX); no longer U$1.PD3(TX)
- net USB_VCC: now also ATMEGA32U4.UVCC, ATMEGA32U4.VBUS, USB_MICROB.VCC; no longer JP3.VCC, U$1.UVCC, U$1.VBUS
Other:
- note added: "ATmega32U4"
- note added: "Active High"
- note added: "Headers"
- note added: "Inputs"
- note added: "Michelle Shorter"
- note added: "Power"
- note added: "XBee"
- moved on the sheet: C1, C2, C3, I2C, JP1, JP2, LED12, LED3, LED34, LED4, LED5, LED6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
